File: CANFD_module.kicad_pcb (KiCad board)
At the start: 2 copper layers, 26.1 x 40.6 mm, 24 parts, among them SW1 SS-12SDP2, U1 MCP2558FD, U2 MCP2517FD, U4 AZ1117CH-3.3TRG1, X1 XRCGB40M000F4M01R0

Commit message: [fix]versionの表示
Other:
- board text added: "ver 2.0"
